File: ADSP-21477_or_21478 breakout/ADSP-21477_or_21478_breakout.brd (EAGLE design)
At the start: 54.7 x 73.9 mm, 20 parts

Commit message: Update DAC,ADC, and ADSP
Routing:
- net N$75: track 50.5 -> 0.00 mm
- net GND: track 134.6 -> 185.1 mm, vias 22 -> 69
- added copper zone on layer 1, net GND
- added copper zone on layer 16, net GND
Other:
- board text added: "ADSP-21477/78 Breakout"
- board text removed: "ADSP-21477/8 Breakout"
Changed lines of the file:
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@@
 <?xml version="1.0" encoding="utf-8"?>
 <!DOCTYPE eagle SYSTEM "eagle.dtd">
-<eagle version="6.3">
+<eagle version="6.5.0">
 <drawing>
 <settings>
@@
 <setting verticaltext="up"/>
 </settings>
-<grid distance="0.025" unitdist="inch" unit="inch" style="lines" multiple="1" display="yes" altdistance="0.025" altunitdist="inch" altunit="inch"/>
+<grid distance="0.1" unitdist="mm" unit="mm" style="lines" multiple="1" display="yes" altdistance="0.025" altunitdist="inch" altunit="inch"/>
 <layers>
 <layer number="1" name="Top" color="4" fill="1" visible="yes" active="yes"/>
@@
 VDD_THD
 3.3V</text>
-<text x="13.97" y="1.905" size="1.4224" layer="20" rot="R90">SHANNON STRUTZ</text>
+<text x="12.505" y="0.83" size="1.778" layer="122">SHANNON STRUTZ</text>
 <hole x="6.35" y="-2.54" drill="3.175"/>
 <hole x="50.8" y="-2.54" drill="3.175"/>
 <hole x="6.35" y="66.04" drill="3.175"/>
-<text x="18.415" y="1.27" size="1.4224" layer="112" rot="R90">ADSP-21477/8 Breakout
-</text>
 <wire x1="46.355" y1="43.18" x2="35.56" y2="43.18" width="0.254" layer="112"/>
 <wire x1="35.56" y1="43.18" x2="35.56" y2="34.29" width="0.254" layer="112"/>
@@
 <hole x="33.02" y="-2.54" drill="3.175"/>
 <hole x="41.91" y="-2.54" drill="3.175"/>
+<text x="13.7" y="11.5" size="1.778" layer="121">ADSP-21477/78
+Breakout</text>
 </plain>
 <attributes>
@@
 <wire x1="30.85" y1="26.15" x2="30.85" y2="24.95" width="0.254" layer="16"/>
 <wire x1="31.7" y1="24.05" x2="30.85" y2="24.9" width="0.254" layer="16"/>
+<polygon width="0.254" layer="16">
+<vertex x="55.9" y="-5.2"/>
+<vertex x="1.2" y="-5.2"/>
+<vertex x="1.2" y="68.7"/>
+<vertex x="55.9" y="68.7"/>
+<vertex x="55.9" y="-5.1"/>
+</polygon>
+<wire x1="28" y1="6.4" x2="25.9" y2="6.4" width="3.81" layer="16"/>
+<wire x1="25.9" y1="6.4" x2="16.2" y2="16.1" width="3.81" layer="16"/>
+<wire x1="16.2" y1="16.1" x2="16.2" y2="25.5" width="3.81" layer="16"/>
+<wire x1="16.2" y1="25.5" x2="18.1" y2="27.4" width="3.81" layer="16"/>
+<wire x1="18.1" y1="27.4" x2="22.8" y2="27.4" width="3.81" layer="16"/>
+<wire x1="22.8" y1="27.4" x2="24.3" y2="27.4" width="3.81" layer="16"/>
+<wire x1="24.3" y1="27.4" x2="25.4" y2="28.5" width="3.81" layer="16"/>
+<wire x1="25.4" y1="28.5" x2="29.4" y2="28.5" width="3.81" layer="16"/>
+<wire x1="29.4" y1="28.5" x2="29.4" y2="25.2" width="3.81" layer="16"/>
+<wire x1="29.4" y1="25.2" x2="25" y2="25.2" width="3.81" layer="16"/>
+<wire x1="25" y1="25.2" x2="22.8" y2="27.4" width="3.81" layer="16"/>
+<polygon width="0.254" layer="1" rank="3">
+<vertex x="1.2" y="-5.2"/>
+<vertex x="55.9" y="-5.2"/>
+<vertex x="55.9" y="68.7"/>
+<vertex x="1.2" y="68.7"/>
+</polygon>
+<via x="23.2" y="62.1" extent="1-16" drill="0.6"/>
+<via x="24.5" y="62.1" extent="1-16" drill="0.6"/>
+<via x="25.8" y="62.1" extent="1-16" drill="0.6"/>
+<via x="27.1" y="62.1" extent="1-16" drill="0.6"/>
+<via x="27.1" y="60.8" extent="1-16" drill="0.6"/>
+<via x="25.8" y="60.8" extent="1-16" drill="0.6"/>
+<via x="25.8" y="59.5" extent="1-16" drill="0.6"/>
+<via x="24.5" y="59.5" extent="1-16" drill="0.6"/>
+<via x="24.5" y="60.8" extent="1-16" drill="0.6"/>
+<via x="23.2" y="60.8" extent="1-16" drill="0.6"/>
+<via x="23.2" y="59.5" extent="1-16" drill="0.6"/>
+<via x="23.2" y="58.2" extent="1-16" drill="0.6"/>
+<via x="24.5" y="58.2" extent="1-16" drill="0.6"/>
+<via x="28.4" y="62.1" extent="1-16" drill="0.6"/>
+<via x="23.2" y="56.9" extent="1-16" drill="0.6"/>
+<via x="11.1" y="28" extent="1-16" drill="0.6"/>
+<via x="11.1" y="25.4" extent="1-16" drill="0.6"/>
+<via x="11.1" y="22.8" extent="1-16" drill="0.6"/>
+<via x="11.1" y="20.3" extent="1-16" drill="0.6"/>
+<via x="7.3" y="2.2" extent="1-16" drill="0.6"/>
+<via x="8.9" y="5" extent="1-16" drill="0.6"/>
+<via x="10" y="7.5" extent="1-16" drill="0.6"/>
+<via x="10" y="10.1" extent="1-16" drill="0.6"/>
+<via x="11.1" y="12.7" extent="1-16" drill="0.6"/>
+<via x="11.1" y="17.8" extent="1-16" drill="0.6"/>
+<via x="11.1" y="15.2" extent="1-16" drill="0.6"/>
+<via x="17.7" y="45.8" extent="1-16" drill="0.6"/>
+<via x="15.2" y="45.8" extent="1-16" drill="0.6"/>
+<via x="12.7" y="45.7" extent="1-16" drill="0.6"/>
+<via x="12.7" y="43.2" extent="1-16" drill="0.6"/>
+<via x="12.7" y="40.6" extent="1-16" drill="0.6"/>
+<via x="47.3" y="28.2" extent="1-16" drill="0.6"/>
+<via x="45.9" y="29.4" extent="1-16" drill="0.6"/>
+<via x="42.1" y="33.2" extent="1-16" drill="0.6"/>
+<via x="43.4" y="32" extent="1-16" drill="0.6"/>
+<via x="44.6" y="30.7" extent="1-16" drill="0.6"/>
+<via x="39.5" y="33.2" extent="1-16" drill="0.6"/>
+<via x="46.2" y="20.6" extent="1-16" drill="0.6"/>
+<via x="46.2" y="12.8" extent="1-16" drill="0.6"/>
+<via x="46.3" y="10.2" extent="1-16" drill="0.6"/>
+<via x="46.3" y="7.7" extent="1-16" drill="0.6"/>
+<via x="46.4" y="2.7" extent="1-16" drill="0.6"/>
+<via x="46.3" y="5.1" extent="1-16" drill="0.6"/>
+<via x="30.5" y="53.4" extent="1-16" drill="0.6"/>
+<via x="37.5" y="65.7" extent="1-16" drill="0.6"/>
+<via x="11.2" y="33.5" extent="1-16" drill="0.6"/>
+<via x="10.7" y="30.3" extent="1-16" drill="0.6"/>
 </signal>
 <signal name="TMS">
@@
 <via x="29.718" y="29.464" extent="1-16" drill="0.3302" diameter="0.254"/>
 </signal>
-<signal name="N$75">
-<wire x1="28" y1="6.4" x2="25.9" y2="6.4" width="3.81" layer="16"/>
-<wire x1="25.9" y1="6.4" x2="16.2" y2="16.1" width="3.81" layer="16"/>
-<wire x1="16.2" y1="16.1" x2="16.2" y2="25.5" width="3.81" layer="16"/>
-<wire x1="16.2" y1="25.5" x2="18.1" y2="27.4" width="3.81" layer="16"/>
-<wire x1="18.1" y1="27.4" x2="22.8" y2="27.4" width="3.81" layer="16"/>
-<wire x1="22.8" y1="27.4" x2="24.3" y2="27.4" width="3.81" layer="16"/>
-<wire x1="24.3" y1="27.4" x2="25.4" y2="28.5" width="3.81" layer="16"/>
-<wire x1="25.4" y1="28.5" x2="29.4" y2="28.5" width="3.81" layer="16"/>
-<wire x1="29.4" y1="28.5" x2="29.4" y2="25.2" width="3.81" layer="16"/>
-<wire x1="29.4" y1="25.2" x2="25" y2="25.2" width="3.81" layer="16"/>
-<wire x1="25" y1="25.2" x2="22.8" y2="27.4" width="3.81" layer="16"/>
-</signal>
 <signal name="N$1">
 <wire x1="25.4635" y1="19.812" x2="25.4635" y2="18.4785" width="0.254" layer="16"/>
@@
 <wire x1="27.7495" y1="19.812" x2="27.7495" y2="18.4785" width="0.254" layer="16"/>
 </signal>
+<signal name="N$5">
+<via x="20.5" y="33.3" extent="1-16" drill="0.6"/>
+</signal>
 </signals>
