File: CS4344 & CS5343/CS5343 ADC/ADC.sch (EAGLE design)
At the start: 21 parts

Commit message: Update DAC,ADC, and ADSP
Connections:
- net N$5 renamed MCLK
- net N$7 renamed LRCLK
- net N$8 renamed SCLK
- net N$9 renamed SOUT
Changed lines of the file:
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@@
 <?xml version="1.0" encoding="utf-8"?>
 <!DOCTYPE eagle SYSTEM "eagle.dtd">
-<eagle version="6.3">
+<eagle version="6.5.0">
 <drawing>
 <settings>
@@
 </segment>
 </net>
-<net name="N$5" class="0">
+<net name="MCLK" class="0">
 <segment>
 <pinref part="JP1" gate="A" pin="2"/>
@@
 </segment>
 </net>
-<net name="N$7" class="0">
+<net name="LRCLK" class="0">
 <segment>
 <pinref part="JP1" gate="A" pin="3"/>
@@
 </segment>
 </net>
-<net name="N$8" class="0">
+<net name="SCLK" class="0">
 <segment>
 <pinref part="JP1" gate="A" pin="4"/>
@@
 </segment>
 </net>
-<net name="N$9" class="0">
+<net name="SOUT" class="0">
 <segment>
 <pinref part="JP1" gate="A" pin="5"/>
