File: Stout IEEE full Dev Board/Stout IEEE full dev board.brd (EAGLE design)
At the start: 74.6 x 55.6 mm, 20 parts, among them J1 POWER_JACKPTH, U1 ARDUINO_SHIELDNO_SILK, U2 V_REG_317SMD

Commit message: Updating design to next revision
Parts:
- removed 16MHZ: (no value), SparkFun-FreqCtrl:HC49U-V
- removed 22PF: 22pF, SparkFun:CAP-PTH-SMALL
- removed ISP: AVR_SPI_PRG_6NS, SparkFun:2X3-NS
- removed JP3: (no value), SparkFun:1X08
- removed JTAG: (no value), pinhead:2X05
- removed LED1: (no value), adafruit:LED3MM
- removed U2: V_REG_317SMD, SparkFun-PowerIC:SOT223
- added C6: 0.1uF, SparkFun-Capacitors:CAP-PTH-SMALL
- added C7, C8: 1.0uF, SparkFun-Capacitors:CAP-PTH-SMALL
- added JP1: USB-B, SparkFun-Connectors:USB-B-PTH
- added JP2: (no value), SparkFun-Connectors:1X06
- added R6: (no value), SparkFun-Resistors:AXIAL-0.4
- added S1: (no value), SparkFun-Electromechanical:TACTILE-PTH
- added U$2, U$3: ZENER, SparkFun-DiscreteSemi:DIODE-ZENER
- added U$4: ARDUINO_UNO_R3_SHIELD, Strutz Electronic Industries:ARDUINO_UNO_R3_SHIELD
- added Y1: 16MHz, SparkFun-FreqCtrl:HC49US
- C1: device 1x05smd:CAP-PTH-SMALL -> SparkFun-Capacitors:CAP-PTH-SMALL
- C2: value 22pF -> (none); device SparkFun:CAP-PTH-SMALL -> SparkFun-Capacitors:CAP-PTH-SMALL
- C3, C4: value (none) -> 1.0uF; device 1x05smd:CAP-PTH-SMALL -> SparkFun-Capacitors:CAP-PTH-SMALL
- C5: value (none) -> 1.0uF; device 1x05smd:CPOL-RADIAL-10UF-25V -> SparkFun-Capacitors:CAP-PTH-SMALL
- J1: value POWER_JACKPTH -> AVR_SPI_PRG_6PTH; device SparkFun:POWER_JACK_PTH -> SparkFun-Connectors:2X3
- R1: value 240 -> 68; device 1x05smd:AXIAL-0.3 -> SparkFun-Resistors:AXIAL-0.4
- R2: value 390 -> 68; device 1x05smd:AXIAL-0.3 -> SparkFun-Resistors:AXIAL-0.4
- R3: value (none) -> 1.7K; device 1x05smd:AXIAL-0.3 -> SparkFun-Resistors:AXIAL-0.4
- U$1: value ATMEGA16 -> ATMEGA16DIP
- U$5: value (none) -> JTAG; device Strutz Electronic Industries:IEEE_LOGO -> Strutz Electronic Industries:JTAG-FPC
- U$6: value (none) -> V_REG_LD1117VXX; device Strutz Electronic Industries:STOUT_S -> SparkFun-PowerIC:78XXL
- U1: value ARDUINO_SHIELDNO_SILK -> TINY85-20-DIP; device SparkFun-Boards:DUEMILANOVE_VIAS -> SparkFun-DigitalIC:DIP08
- moved C1 71.6 mm to (48.0, 41.1), turned to 270 degrees
- moved J1 64.2 mm to (55.6, 32.5), turned to 90 degrees
- moved C4 62.9 mm to (38.9, 37.6), turned to 90 degrees
- moved U$5 57.9 mm to (3.81, 15.7), turned to 270 degrees
- moved U$6 42.0 mm to (11.9, 5.08), turned to 180 degrees
- moved R2 33.2 mm to (19.8, 36.1), turned to 180 degrees
- moved R1 32.7 mm to (19.8, 39.1), turned to 180 degrees
- moved R3 28.0 mm to (19.6, 44.2), turned to 180 degrees
- moved C3 22.3 mm to (5.84, 25.4), turned to 180 degrees
- moved C2 21.8 mm to (48.0, 33.3), turned to 90 degrees
- moved U1 18.8 mm to (31.8, 38.1), turned to 0 degrees
- moved U$1 15.5 mm to (33.5, 20.6), turned to 270 degrees
- moved C5 12.0 mm to (4.06, 8.89)
Connections:
- removed net N$13: U$1.14, U1.RX
- removed net N$14: U$1.15, U1.TX
- removed net N$15: U$1.16, U1.D2
- removed net N$16: U$1.17, U1.D3
- removed net N$17: 16MHZ.2, C2.1, U$1.13
- removed net N$18: 16MHZ.1, 22PF.1, U$1.12
- removed net N$19: JP3.6, U$1.23
- removed net N$20: JP3.5, U$1.22
- removed net N$21: U$1.1, U1.D4
- removed net N$22: U$1.20, U1.D8
- removed net N$23: LED1.A, R3.P$2
- removed net N$24: U$1.5, U1.D10
- removed net N$25: U$1.2, U1.D5
- removed net N$26: U$1.19, U1.D9
- removed net N$27: U$1.4, U1.D7
- removed net N$28: U$1.3, U1.D6
- removed net N$29: JTAG.1, U$1.24
- removed net N$3: U$1.38, U1.A2
- removed net N$30: JTAG.3, U$1.26
- removed net N$31: JTAG.5, U$1.25
- removed net N$32: JTAG.9, U$1.27
- removed net N$33: JP3.2, U$1.21
- removed net N$34: JP3.1, U$1.18
- removed net N$35: JP3.4, U$1.28
- removed net N$36: JP3.3, U$1.29
- removed net N$6: U$1.35, U1.A5
- removed net N$7: R1.P$2, U1.3.3V, U2.2
- removed net N$9: JP3.7, U$1.34
- removed net RESET: ISP.5, JTAG.6, U$1.9, U1.RES
- new net 3.3V: C7.2, U$4.3.3V, U$6.GND
- new net ADC0: U$1.40, U$4.A0
- new net ADC1: U$1.39, U$4.A1
- new net ADC2: U$1.38, U$4.A2
- new net ADC3: U$1.37, U$4.A3
- new net ADC4: U$1.36, U$4.A4
- new net ADC5: U$1.35, U$4.A5
- new net AREF: U$1.32, U$4.AREF
- new net D2: U$1.16, U$4.D2
- new net D3: U$1.17, U$4.D3
- new net D4: U$1.1, U$4.D4
- new net D5: U$1.2, U$4.D5
- new net D6: U$1.3, U$4.D6
- new net D7: U$1.4, U$4.D7
- new net D8: U$1.20, U$4.D8
- new net D9: U$1.19, U$4.D9
- new net EB1: JP2.1, U$1.18
- new net EB2: JP2.2, U$1.21
- new net EB3: JP2.3, U$1.28
- new net EB4: JP2.4, U$1.29
- new net EB5: JP2.5, U$1.33
- new net EB6: JP2.6, U$1.34
- new net RX: U$1.14, U$4.RX
- new net SCL: U$1.22, U$4.SCL
- new net SDA: U$1.23, U$4.SDA
- new net SS: U$1.5, U$4.D10
- new net TX: U$1.15, U$4.TX
- new net USB-D_N: R1.P$1, U1.3
- new net USB-D_P: R2.P$1, U1.2
- new net ~RESET: J1.5, R6.P$2, S1.3, S1.4, U$1.9, U$4.RES, U1.1
- net GND: now also C1.1, C2.1, C3.1, C4.1, C5.1, C6.1, C7.1, C8.1, J1.6, JP1.GND, S1.1, S1.2, U$2.P$2, U$3.P$2, U$4.GND@0, U$4.GND@1, U$4.GND@2, U$5.1, U$6.IN, U1.4; no longer 22PF.2, C1.2, C2.2, C3.2, C4.2, C5.2, ISP.6, J1.GND, J1.GNDBREAK, JTAG.10, JTAG.2, LED1.K, R2.P$1, U1.GND@0, U1.GND@1, U1.GND@2
- net MISO: now also J1.1, U$4.D12, U1.6; no longer ISP.1, U1.D12
- net MOSI: now also J1.4, U$4.D11, U1.5; no longer ISP.4, U1.D11
- net N$1: now also C2.2, U$1.12, Y1.1; no longer U$1.40, U1.A0
- net N$10: now also U$1.25, U$5.5; no longer R1.P$1, R2.P$2, U2.1
- net N$11: now also U$1.26, U$5.4; no longer U$1.32, U1.AREF
- net N$12: now also U$1.27, U$5.3; no longer C1.1, C5.1, J1.PWR, R3.P$1, U1.VIN, U2.3
- net N$2: now also C1.2, U$1.13, Y1.2; no longer U$1.39, U1.A1
- net N$4: now also JP1.D-, R1.P$2, R3.P$2, U$2.P$1; no longer U$1.37, U1.A3
- net N$5: now also JP1.D+, R2.P$2, U$3.P$1; no longer U$1.36, U1.A4
- net N$8: now also U$1.24, U$5.2; no longer JP3.8, U$1.33
- net SCK: now also J1.3, U$4.D13, U1.7; no longer ISP.3, U1.D13
- net VCC: now also C3.2, C4.2, C5.2, C6.2, C8.2, J1.2, JP1.VBUS, R6.P$1, U$4.5V, U$5.6, U$6.OUT, U1.8; no longer C3.1, C4.1, ISP.2, JTAG.4, JTAG.7, U1.5V
Routing:
- net GND: track 186.0 -> 4.13 mm, vias 1 -> 0
- net N$29: track 116.1 -> 0.00 mm, vias 5 -> 0
- net VCC: track 123.6 -> 8.54 mm, vias 4 -> 0
- net ~RESET: track 0.00 -> 112.4 mm, vias 0 -> 5
- net RESET: track 96.8 -> 0.00 mm, vias 1 -> 0
- net N$31: track 80.9 -> 0.00 mm, vias 5 -> 0
- net MISO: track 126.8 -> 49.7 mm, vias 2 -> 0
- net N$24: track 74.5 -> 0.00 mm, vias 4 -> 0
- net N$6: track 67.0 -> 0.00 mm
- net N$3: track 64.7 -> 0.00 mm
- net N$9: track 60.0 -> 0.00 mm, vias 5 -> 0
- net N$28: track 59.1 -> 0.00 mm, vias 1 -> 0
- net N$5: track 66.4 -> 9.75 mm
- net N$4: track 65.6 -> 9.61 mm
- net AREF: track 0.00 -> 55.8 mm, vias 0 -> 2
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- added copper zone on layer 16, net GND
- added copper zone on layer 1, net VCC
Other:
- board size 74.6 x 55.6 mm -> 59.7 x 53.3 mm
- board text added: "2015"
- board text added: "Designed by: Shannon Strutz"
- board text added: "University of Wisconsin - Stout"
- board text removed: "2013"
- board text removed: "Designed by Shannon Strutz"
- board text removed: "GND"
- board text removed: "UW-Stout"
- board text removed: "for University of Wisconsin - Stout"
