File: Stout IEEE full Dev Board/Stout IEEE full dev board.sch (EAGLE design)
At the start: 18 parts, among them J1 POWER_JACKPTH, U1 ARDUINO_SHIELDNO_SILK, U2 V_REG_317SMD

Commit message: Updating design to next revision
Parts:
- removed 16MHZ: (no value), SparkFun-FreqCtrl:CRYSTALHC49UV
- removed 22PF: 22pF, SparkFun:CAPPTH
- removed ISP: AVR_SPI_PRG_6NS, SparkFun:AVR_SPI_PRG_6NS
- removed JP3: (no value), SparkFun:M08
- removed JTAG: (no value), pinhead:PINHD-2X5
- removed LED1: (no value), adafruit:LED3MM
- removed U2: V_REG_317SMD, SparkFun-PowerIC:V_REG_317SMD
- added C6: 0.1uF, SparkFun-Capacitors:CAPPTH
- added C7, C8: 1.0uF, SparkFun-Capacitors:CAPPTH
- added JP1: USB-B, SparkFun-Connectors:USBPTH
- added JP2: (no value), SparkFun-Connectors:M06SIP
- added R6: (no value), SparkFun-Resistors:RESISTORPTH-1/4W
- added S1: (no value), SparkFun-Electromechanical:TAC_SWITCHPTH
- added U$2, U$3: ZENER, SparkFun-DiscreteSemi:DIODE-ZENERPTH
- added U$4: ARDUINO_UNO_R3_SHIELD, Strutz Electronic Industries:ARDUINO_UNO_R3_SHIELD
- added U$5: JTAG, Strutz Electronic Industries:JTAG
- added U$6: V_REG_LD1117VXX, SparkFun-PowerIC:V_REG_LD1117VXX
- added Y1: 16MHz, SparkFun-FreqCtrl:CRYSTALHC49US
- C1: device 1x05smd:CAPPTH -> SparkFun-Capacitors:CAPPTH
- C2: value 22pF -> (none); device SparkFun:CAPPTH -> SparkFun-Capacitors:CAPPTH
- C3, C4: value (none) -> 1.0uF; device 1x05smd:CAPPTH -> SparkFun-Capacitors:CAPPTH
- C5: value (none) -> 1.0uF; device 1x05smd:CAP_POLPTH2 -> SparkFun-Capacitors:CAPPTH
- J1: value POWER_JACKPTH -> AVR_SPI_PRG_6PTH; device SparkFun:POWER_JACKPTH -> SparkFun-Connectors:AVR_SPI_PRG_6PTH
- R1: value 240 -> 68; device 1x05smd:RESISTORPTH1 -> SparkFun-Resistors:RESISTORPTH-1/4W
- R2: value 390 -> 68; device 1x05smd:RESISTORPTH1 -> SparkFun-Resistors:RESISTORPTH-1/4W
- R3: value (none) -> 1.7K; device 1x05smd:RESISTORPTH1 -> SparkFun-Resistors:RESISTORPTH-1/4W
- U$1: value ATMEGA16 -> ATMEGA16DIP; device Strutz Electronic Industries:ATMEGA16 -> Strutz Electronic Industries:ATMEGA16DIP
- U1: value ARDUINO_SHIELDNO_SILK -> TINY85-20-DIP; device SparkFun-Boards:ARDUINO_SHIELDNO_SILK -> SparkFun-DigitalIC:ATTINY45TINY85-20-DIP
Connections:
- removed net N$13: U$1.PD0(RXD), U1.RX
- removed net N$14: U$1.PD1(TXD), U1.TX
- removed net N$15: U$1.PD2(INT0), U1.D2
- removed net N$16: U$1.PD3(INT1), U1.*D3
- removed net N$17: 16MHZ.2, C2.1, U$1.XTAL1
- removed net N$18: 16MHZ.1, 22PF.1, U$1.XTAL2
- removed net N$19: JP3.6, U$1.PC1(SDA)
- removed net N$20: JP3.5, U$1.PC0(SCL)
- removed net N$21: U$1.PB0(XCK/T0), U1.D4
- removed net N$22: U$1.PD6(ICP1), U1.D8
- removed net N$23: LED1.A, R3.2
- removed net N$24: U$1.PB4(~SS), U1.*D10
- removed net N$25: U$1.PB1(T1), U1.*D5
- removed net N$26: U$1.PD5(OC1A), U1.*D9
- removed net N$27: U$1.PB3(OC0/AIN1), U1.D7
- removed net N$28: U$1.PB2(INT2/AIN0), U1.*D6
- removed net N$29: JTAG.1, U$1.PC2(TCK)
- removed net N$3: U$1.PA2(ADC2), U1.A2
- removed net N$30: JTAG.3, U$1.PC4(TDO)
- removed net N$31: JTAG.5, U$1.PC3(TMS)
- removed net N$32: JTAG.9, U$1.PC5(TDI)
- removed net N$33: JP3.2, U$1.PD7(OC2)
- removed net N$34: JP3.1, U$1.PD4(OC1B)
- removed net N$35: JP3.4, U$1.PC6(TOSC1)
- removed net N$36: JP3.3, U$1.PC7(TOSC2)
- removed net N$6: U$1.PA5(ADC5), U1.A5
- removed net N$7: R1.2, U1.3.3V, U2.OUT
- removed net N$9: JP3.7, U$1.PA6(ADC6)
- removed net RESET: ISP.5, JTAG.6, U$1.~RESET, U1.RES
- new net 3.3V: C7.2, U$4.3.3V, U$6.OUT
- new net ADC0: U$1.PA0(ADC0), U$4.A0
- new net ADC1: U$1.PA1(ADC1), U$4.A1
- new net ADC2: U$1.PA2(ADC2), U$4.A2
- new net ADC3: U$1.PA3(ADC3), U$4.A3
- new net ADC4: U$1.PA4(ADC4), U$4.A4
- new net ADC5: U$1.PA5(ADC5), U$4.A5
- new net AREF: U$1.AREF, U$4.AREF
- new net D2: U$1.PD2(INT0), U$4.D2
- new net D3: U$1.PD3(INT1), U$4.*D3
- new net D4: U$1.PB0(XCK/T0), U$4.D4
- new net D5: U$1.PB1(T1), U$4.*D5
- new net D6: U$1.PB2(INT2/AIN0), U$4.*D6
- new net D7: U$1.PB3(OC0/AIN1), U$4.D7
- new net D8: U$1.PD6(ICP1), U$4.D8
- new net D9: U$1.PD5(OC1A), U$4.*D9
- new net EB1: JP2.1, U$1.PD4(OC1B)
- new net EB2: JP2.2, U$1.PD7(OC2)
- new net EB3: JP2.3, U$1.PC6(TOSC1)
- new net EB4: JP2.4, U$1.PC7(TOSC2)
- new net EB5: JP2.5, U$1.PA7(ADC7)
- new net EB6: JP2.6, U$1.PA6(ADC6)
- new net RX: U$1.PD0(RXD), U$4.RX
- new net SCL: U$1.PC0(SCL), U$4.SCL
- new net SDA: U$1.PC1(SDA), U$4.SDA
- new net SS: U$1.PB4(~SS), U$4.*D10
- new net TX: U$1.PD1(TXD), U$4.TX
- new net USB-D_N: R1.1, U1.PB4(ADC2)
- new net USB-D_P: R2.1, U1.PB3(ADC3)
- new net ~RESET: J1.5, R6.2, S1.3, S1.4, U$1.~RESET, U$4.RES, U1.PB5(NRES)
- net GND: now also C1.1, C2.1, C3.1, C4.1, C5.1, C6.1, C7.1, C8.1, J1.6, JP1.GND, S1.1, S1.2, U$2.A, U$3.A, U$4.GND@0, U$4.GND@1, U$4.GND@2, U$5.GND, U$6.GND, U1.GND; no longer 22PF.2, C1.2, C2.2, C3.2, C4.2, C5.-, ISP.6, J1.GND, J1.GNDBREAK, JTAG.10, JTAG.2, LED1.C, R2.1, U1.GND@0, U1.GND@1, U1.GND@2
- net MISO: now also J1.1, U$4.D12, U1.PB1(MISO); no longer ISP.1, U1.D12
- net MOSI: now also J1.4, U$4.*D11, U1.PB0(MOSI); no longer ISP.4, U1.*D11
- net N$1: now also C2.2, U$1.XTAL2, Y1.1; no longer U$1.PA0(ADC0), U1.A0
- net N$10: now also U$1.PC3(TMS), U$5.TMS; no longer R1.1, R2.2, U2.ADJ
- net N$11: now also U$1.PC4(TDO), U$5.TDO; no longer U$1.AREF, U1.AREF
- net N$12: now also U$1.PC5(TDI), U$5.TDI; no longer C1.1, C5.+, J1.PWR, R3.1, U1.VIN, U2.IN
- net N$2: now also C1.2, U$1.XTAL1, Y1.2; no longer U$1.PA1(ADC1), U1.A1
- net N$4: now also JP1.D-, R1.2, R3.2, U$2.C; no longer U$1.PA3(ADC3), U1.A3
- net N$5: now also JP1.D+, R2.2, U$3.C; no longer U$1.PA4(ADC4), U1.A4
- net N$8: now also U$1.PC2(TCK), U$5.TCK; no longer JP3.8, U$1.PA7(ADC7)
- net SCK: now also J1.3, U$4.D13, U1.PB2(SCK/ADC1); no longer ISP.3, U1.D13
- net VCC: now also C3.2, C4.2, C5.2, C6.2, C8.2, J1.2, JP1.VBUS, R6.1, U$4.5V, U$5.VCC, U$6.IN, U1.VCC; no longer C3.1, C4.1, ISP.2, JTAG.4, JTAG.7, U1.5V
Other:
- moved on the sheet: C1, C2, C3, C4, R1, R2, R3
